File: Hardware/Shields/PiShield/Pi.brd (EAGLE design)
At the start: 58 x 56 mm, 6 parts, among them IC2 MAX3082

Commit message: Bilag added KE
Parts:
- moved C5 10.8 mm to (12.5, 8.33)
- moved R7 7.07 mm to (35.6, 18.2)
- moved R6 7.00 mm to (37.3, 15.2)
- moved IC2 6.08 mm to (22.4, 12.1), turned to 90 degrees
Routing:
- net GND: track 0.00 -> 60.9 mm
- net OE_DIFF-: track 0.00 -> 60.0 mm
- net OE_DIFF+: track 0.00 -> 40.8 mm, vias 0 -> 1
- net KAR_TX: track 0.00 -> 29.0 mm
- net KAR_RX: track 0.00 -> 26.0 mm
- net OE_TX_ENA: track 0.00 -> 8.30 mm
- net N$1: track 0.00 -> 3.75 mm, vias 0 -> 1
- net VCC: track 0.00 -> 3.49 mm
- net N$3: track 0.00 -> 2.64 mm, vias 0 -> 1
