File: Hardware/Shields/KarShield/KarShield.sch (EAGLE design)
At the start: 42 parts, among them IC1 MAX3082, IC2 MAX3082

Commit message: Shields KE
Parts:
- added 12V: (no value), con-phoenix-254:MPT2
Connections:
- removed net +5V: 74HC08.VCC, 74HC393.VCC, FS-1.1, S1.S
- removed net I_VALVE_T1: C1.1, D1.C, I_VALVE-1.1
- removed net KAR_GND: IC1.GND, KAR_BUS-3.1, R4.1
- removed net O_VALVE_T1: C2.1, D2.C
- removed net PUMP_T1_VCC: C3.1, D3.C, PUMP-1.1
- removed net VCC: C4.1, C5.1, C6.1, IC1.VCC, IC2.VCC, R8.2
- new net 12V: 12V-2.1, C1.1, C2.1, C3.1, D1.C, D2.C, D3.C, I_VALVE-1.1, PUMP-1.1
- new net 5V: 74HC08.VCC, 74HC393.VCC, C4.1, C5.1, C6.1, FS-1.1, IC1.VCC, IC2.VCC, R8.2, S1.S
- net GND: now also 12V-1.1, IC1.GND, KAR_BUS-3.1, PUMP-2.1, R4.1
- net PUMP_T2_GND: no longer PUMP-2.1
